Commit message: Cleaned up code

File: src/inverse_kinematics_pkg/urdf/puma.urdf (robot description, URDF)
Before this commit: robot puma, 8 links, 7 joints
Links:
- link link4: geometry visual cylinder length=0.2 radius=0.05
- link link5: geometry visual cylinder length=0.2 radius=0.05
- link link6: geometry visual sphere radius=0.05
Joints:
- joint map_to_base: axis 0 0 1 -> (none)
